File: Amiga-A1012.sch (KiCad schematic (older format))
At the start: 10 parts, among them U1 74LS38, U2 74LS74, U3 74LS38

Commit message: Added decoupling caps. More routing.
Parts:
- added C4, C5, C6: 100nF, Resistors_SMD:R_0603, symbol C
Connections:
- net +5V: now also C5.1
- net GND: now also C5.2
- new net: C4.1, C6.1
- new net: C4.2, C6.2
Changed lines of the file:
@@
 	1    0    0    -1
 $EndComp
+$Comp
+L C C4
+U 1 1 5900EDD9
+P 3500 7100
+F 0 "C4" H 3525 7200 50  0000 L CNN
+F 1 "100nF" H 3525 7000 50  0000 L CNN
+F 2 "Resistors_SMD:R_0603" H 3538 6950 50  0001 C CNN
+F 3 "" H 3500 7100 50  0000 C CNN
+	1    3500 7100
+	1    0    0    -1
+$EndComp
+$Comp
+L C C5
+U 1 1 5900EF38
+P 3800 7100
+F 0 "C5" H 3825 7200 50  0000 L CNN
+F 1 "100nF" H 3825 7000 50  0000 L CNN
+F 2 "Resistors_SMD:R_0603" H 3838 6950 50  0001 C CNN
+F 3 "" H 3800 7100 50  0000 C CNN
+	1    3800 7100
+	1    0    0    -1
+$EndComp
+$Comp
+L C C6
+U 1 1 5900EF7B
+P 4100 7100
+F 0 "C6" H 4125 7200 50  0000 L CNN
+F 1 "100nF" H 4125 7000 50  0000 L CNN
+F 2 "Resistors_SMD:R_0603" H 4138 6950 50  0001 C CNN
+F 3 "" H 4100 7100 50  0000 C CNN
+	1    4100 7100
+	1    0    0    -1
+$EndComp
+$Comp
+L +5V #PWR014
+U 1 1 5900EFB4
+P 3800 6950
+F 0 "#PWR014" H 3800 6800 50  0001 C CNN
+F 1 "+5V" H 3800 7090 50  0000 C CNN
+F 2 "" H 3800 6950 50  0000 C CNN
+F 3 "" H 3800 6950 50  0000 C CNN
+	1    3800 6950
+	1    0    0    -1
+$EndComp
+$Comp
+L GND #PWR015
+U 1 1 5900EFEC
+P 3800 7250
+F 0 "#PWR015" H 3800 7000 50  0001 C CNN
+F 1 "GND" H 3800 7100 50  0000 C CNN
+F 2 "" H 3800 7250 50  0000 C CNN
+F 3 "" H 3800 7250 50  0000 C CNN
+	1    3800 7250
+	1    0    0    -1
+$EndComp
+Wire Wire Line
+	3500 6950 4100 6950
+Wire Wire Line
+	3500 7250 4100 7250
 $EndSCHEMATC

Commit message: More routing. Connected VCC to +5V net, for LS chips.
Connections:
- net +5V: now also C4.1, C6.1
- net GND: now also C4.2, C6.2
Changed lines of the file:
@@
 Wire Wire Line
 	3500 7250 4100 7250
+$Comp
+L +5V #PWR?
+U 1 1 5902272D
+P 1100 4400
+F 0 "#PWR?" H 1100 4250 50  0001 C CNN
+F 1 "+5V" H 1100 4540 50  0000 C CNN
+F 2 "" H 1100 4400 50  0000 C CNN
+F 3 "" H 1100 4400 50  0000 C CNN
+	1    1100 4400
+	1    0    0    -1
+$EndComp
+$Comp
+L VCC #PWR?
+U 1 1 590227AD
+P 1300 4400
+F 0 "#PWR?" H 1300 4250 50  0001 C CNN
+F 1 "VCC" H 1300 4550 50  0000 C CNN
+F 2 "" H 1300 4400 50  0000 C CNN
+F 3 "" H 1300 4400 50  0000 C CNN
+	1    1300 4400
+	1    0    0    -1
+$EndComp
+Wire Wire Line
+	1100 4400 1300 4400
+Connection ~ 3800 7250
+Connection ~ 3800 6950
 $EndSCHEMATC

Commit message: Finished routing. Fixed routing problems with unconnected nets. Added fiducials.
Changed lines of the file:
@@
 L +5V #PWR?
 U 1 1 5902272D
-P 1100 4400
-F 0 "#PWR?" H 1100 4250 50  0001 C CNN
-F 1 "+5V" H 1100 4540 50  0000 C CNN
-F 2 "" H 1100 4400 50  0000 C CNN
-F 3 "" H 1100 4400 50  0000 C CNN
-	1    1100 4400
+P 4700 3850
+F 0 "#PWR?" H 4700 3700 50  0001 C CNN
+F 1 "+5V" H 4700 3990 50  0000 C CNN
+F 2 "" H 4700 3850 50  0000 C CNN
+F 3 "" H 4700 3850 50  0000 C CNN
+	1    4700 3850
+	1    0    0    -1
+$EndComp
+Connection ~ 3800 7250
+Connection ~ 3800 6950
+$Comp
+L GND #PWR?
+U 1 1 5904D074
+P 3400 4100
+F 0 "#PWR?" H 3400 3850 50  0001 C CNN
+F 1 "GND" H 3400 3950 50  0000 C CNN
+F 2 "" H 3400 4100 50  0000 C CNN
+F 3 "" H 3400 4100 50  0000 C CNN
+	1    3400 4100
 	1    0    0    -1
 $EndComp
 $Comp
-L VCC #PWR?
-U 1 1 590227AD
-P 1300 4400
-F 0 "#PWR?" H 1300 4250 50  0001 C CNN
-F 1 "VCC" H 1300 4550 50  0000 C CNN
-F 2 "" H 1300 4400 50  0000 C CNN
-F 3 "" H 1300 4400 50  0000 C CNN
-	1    1300 4400
+L GND #PWR?
+U 1 1 5904D226
+P 3400 5650
+F 0 "#PWR?" H 3400 5400 50  0001 C CNN
+F 1 "GND" H 3400 5500 50  0000 C CNN
+F 2 "" H 3400 5650 50  0000 C CNN
+F 3 "" H 3400 5650 50  0000 C CNN
+	1    3400 5650
 	1    0    0    -1
 $EndComp
-Wire Wire Line
-	1100 4400 1300 4400
-Connection ~ 3800 7250
-Connection ~ 3800 6950
+$Comp
+L GND #PWR?
+U 1 1 5904D312
+P 4700 4350
+F 0 "#PWR?" H 4700 4100 50  0001 C CNN
+F 1 "GND" H 4700 4200 50  0000 C CNN
+F 2 "" H 4700 4350 50  0000 C CNN
+F 3 "" H 4700 4350 50  0000 C CNN
+	1    4700 4350
+	1    0    0    -1
+$EndComp
 $EndSCHEMATC

Commit message: Work in progress, fixing problems found in prototype:  * swapped clock and data on LS74  * need pull-up on LS38 to LS74  * add pull-ups on unused LS38 gates  * connect drive reset
Started to reduce size.
Parts:
- added R2, R3, R4, R5: 1K, Resistors_SMD:R_0603, symbol R_Small
- added unit 4 of U1
- added unit 4 of U3
- C1, C2, C3: value 1000µF -> 470µF/10V; footprint Capacitors_SMD:c_elec_10x10.5 -> Capacitors_Tantalum_SMD:Tantalum_Case-D_EIA-7343-31_Reflow
- R1: value 4K7 -> 1K
Connections:
- net +5V: now also R2.1, R3.1, R4.1, R5.1, U1.14 (VCC), U3.14 (VCC)
- net GND: now also U1.7 (GND), U3.7 (GND)
- net at CONN1.10 (/Reset): now also U2.10 (Sd), U2.4 (Sd)
- net at R1.2, U2.1 (Cd), U2.13 (Cd): no longer U2.10 (Sd), U2.4 (Sd)
- net at U1.3, U1.4: now also U2.3 (Cp), R4.2; no longer U2.2 (D)
- net at U3.3, U3.4: now also U2.11 (Cp), R5.2; no longer U2.12 (D)
- new net: CONN1.8 (/Motor), U2.12 (D), U2.2 (D)
- new net: R2.2, U1.12, U1.13
- new net: R3.2, U3.12, U3.13
- no-connect marks 13 -> 14
Other:
- moved on the sheet: R1, U1A, U3A
